Commit message: made imu description visible but need to make it dynamic

File: src/imu_description/urdf/imu_model.urdf.xacro (robot description, xacro)
@@ -5,5 +5,5 @@
     <origin xyz="0 0 0" rpy="0 0 0"/>
     <geometry>
-       <box size="0.03 0.03 0.03"/>
+       <box size="0.3 0.3 0.3"/>
     </geometry>
     <material name="gray">
@@ -12,5 +12,5 @@
    </visual>
   </link>
-  <joint name="base_to_imu" type="fixed">
+  <joint name="base_to_imu" type="floating">
     <origin xyz="0 0 0.03" rpy="0 0 0"/>
     <parent link="base_link"/>
@@ -21,5 +21,5 @@
      <origin xyz="0 0 0" rpy="0 0 0"/>
       <geometry>
-        <box size="0.05 0.05 0.02"/>  <!-- small cube -->
+        <box size="0.5 0.5 0.2"/>  <!-- small cube -->
       </geometry>
       <material name="green">
